File: Trump Card.kicad_sch (KiCad schematic)
At the start: 76 parts, among them J1 Conn_02x05_Odd_Even, P1 Bus_ISA_8bit, U1 Z8001P, U10 6116, U11 PHYSNOCT_PHYSNOCT, U12 74LS245, U13 74LS245, U2 CY62157ELL-45ZSXI, U3 ATF1504-100A, U4 74LS373, U5 74LS373, U6 74LS373, U7 2716, U8 2716, U9 Z8581, Y1 20 MHz

Commit message: Changed CPLD to a EPM7128STC100-15
The new CPLD has more available pins than the Atmel chip, and the programmer is more common and cheaper.
Parts:
- removed U3: ATF1504-100A, Package_QFP:TQFP-100_14x14mm_P0.5mm, symbol cpu-mem4-rescue:ATF1504-100A-cpu-mem4-eagle-import
- removed U4: 74LS373, Package_DIP:DIP-20_W7.62mm, symbol 74xx:74HC373
- added U3: EPM7128STC100-15, libs:QFP50P1600X1600X120-100N, symbol EPM7128STC100-15:EPM7128STC100-15
- Y1: value 20 MHz -> 12 MHz
Connections:
- net +5V: now also U3.11 (GNDIO_3), U3.18 (VCCIO_4), U3.26 (GNDIO), U3.3 (VCCIO_2), U3.34 (VCCIO_5), U3.38 (GNDINT), U3.39 (VCCINT), U3.43 (GNDIO_2), U3.51 (VCCIO), U3.59 (GNDIO_5), U3.66 (VCCIO_6), U3.74 (GNDIO_6), U3.82 (VCCIO_3), U3.86 (GNDINT_2), U3.91 (VCCINT_2), U3.95 (GNDIO_4)
- net AS: now also U3.33 (IO_21)
- net BA0: now also U3.97 (IO_67)
- net BA1: now also U3.98 (IO_68)
- net BA10: now also U3.25 (IO)
- net BA2: now also U3.99 (IO_69)
- net BA3: now also U3.100 (IO_70)
- net BA4: now also U3.19 (IO_71)
- net BA5: now also U3.20 (IO_72)
- net BA6: now also U3.21 (IO_73)
- net BA7: now also U3.22 (IO_74)
- net BA8: now also U3.23 (IO_75)
- net BA9: now also U3.24 (IO_76)
- net BnW: now also U3.37 (IO_24)
- net LA0: now also U3.93 (IO_64)
- net LA1: now also U3.94 (IO_65)
- net LS0: now also U3.13 (IO_11)
- net LS1: now also U3.12 (IO_10)
- net LS2: now also U3.10 (IO_9)
- net LS3: now also U3.9 (IO_8)
- net OSC: now also U3.87 (INPUT/GCLK1)
- net PCA0: now also U3.65 (IO_46)
- net PCA1: now also U3.67 (IO_47)
- net PCA2: now also U3.68 (IO_48)
- net PCA3: now also U3.69 (IO_49)
- net PCA4: now also U3.70 (IO_50)
- net PCA5: now also U3.71 (IO_51)
- net PCA6: now also U3.72 (IO_52)
- net PCA7: now also U3.75 (IO_53)
- net PCA8: now also U3.76 (IO_54)
- net PCA9: now also U3.77 (IO_55)
- net PCD0: now also U3.64 (IO_45)
- net RAMnPROM: now also U3.28 (IO_16)
- net RnW: now also U3.40 (IO_25)
- net SN0: now also U3.58 (IO_41)
- net SN1: now also U3.57 (IO_40)
- net SN2: now also U3.56 (IO_39)
- net SN3: now also U3.55 (IO_38)
- net SN4: now also U3.54 (IO_37)
- net SN5: now also U3.53 (IO_36)
- net SN6: now also U3.52 (IO_35)
- net ST0: now also U3.27 (IO_15)
- net ST1: now also U3.17 (IO_14)
- net ST2: now also U3.16 (IO_13)
- net ST3: now also U3.14 (IO_12)
- net TCK: now also U3.62 (IO/TCK)
- net TDI: now also U3.4 (IO/TDI)
- net TDO: now also U3.73 (IO/TDO)
- net TMS: now also U3.15 (IO/TMS)
- net /AEN: now also U3.60 (IO_42)
- net /AS: now also U3.35 (IO_22)
- net /BHE: now also U3.31 (IO_19)
- net /BLE: now also U3.32 (IO_20)
- net /CS_2716: now also U3.48 (IO_32)
- net /CS_RAM: now also U3.49 (IO_33)
- net /DS: now also U3.36 (IO_23)
- net /HOLD: now also U3.44 (IO_28)
- net /IOR: now also U3.61 (IO_43)
- net /IOW: now also U3.63 (IO_44)
- net /MRD: now also U3.29 (IO_17)
- net /MREQ: now also U3.41 (IO_26)
- net /MWR: now also U3.30 (IO_18)
- net /NMI: now also U3.85 (IO_62)
- net /OE_6116: now also U3.45 (IO_29)
- net /PC: now also U3.46 (IO_30)
- net /RESET: now also U3.92 (IO_63)
- net /WE: now also U3.42 (IO_27)
- net /Z: now also U3.47 (IO_31)
- net /ADDR2: now reaches U9.7 (/ADDR2)
- net /ADDR2: now also U3.50 (IO_34)
- net RESET renamed RESET_DRV
- net RESET_DRV: now also U3.89 (INPUT/*GCLR)
- no-connect marks 65 -> 46
Other:
- moved on the sheet: R22, R23, R24, R25, U10A, U9B, Y1

Commit message: Final commit for V1
Modified the schematic and CPLD assignation to make PCB routing easier,
PCB completed and gerber files provided.
Parts:
- added unit 2 of U4
- P1: footprint pcb:PC-XT-Long -> pcb:PC-XT-Short-6in
- U3: footprint libs:QFP50P1600X1600X120-100N -> Web:QFP50P1600X1600X120-100N
- renumbered U10 to U4
Connections:
- net +5V: now also U4.24 (VCC); no longer C1.2, C10.2, C11.2, C12.2, C13.2, C14.2, C15.2, C16.2, C17.2, C18.2, C19.2, C2.2, C20.2, C21.2, C22.2, C23.2, C24.2, C3.2, C4.2, C5.2, C6.2, C7.2, C8.2, C9.2, J1.10 (Pin_10), J1.2 (Pin_2), P1.B1 (GND), P1.B10 (GND), P1.B31 (GND), TEST-PDS1.2 (Pin_2), TEST-PDS2.2 (Pin_2), U1.36 (GND), U12.10 (GND), U13.10 (GND), U2.12 (VSS), U2.34 (VSS), U3.11 (GNDIO_3), U3.26 (GNDIO), U3.38 (GNDINT), U3.43 (GNDIO_2), U3.59 (GNDIO_5), U3.74 (GNDIO_6), U3.86 (GNDINT_2), U3.95 (GNDIO_4), U5.1 (OE), U5.10 (GND), U6.1 (OE), U6.10 (GND), U7.12 (GND), U8.12 (GND), U9.14 (GND), U9.4 (/INH)
- net AS: now also U3.54 (IO_37); no longer U3.33 (IO_21)
- net BA0: now also U3.32 (IO_20); no longer U3.97 (IO_67)
- net BA1: now also U3.35 (IO_22); no longer U3.98 (IO_68)
- net BA10: now also U3.40 (IO_25); no longer U3.25 (IO)
- net BA2: now also U3.37 (IO_24); no longer U3.99 (IO_69)
- net BA3: now also U3.41 (IO_26); no longer U3.100 (IO_70)
- net BA4: now also U3.44 (IO_28); no longer U3.19 (IO_71)
- net BA5: now also U3.46 (IO_30); no longer U3.20 (IO_72)
- net BA6: now also U3.48 (IO_32); no longer U3.21 (IO_73)
- net BA7: now also U3.50 (IO_34); no longer U3.22 (IO_74)
- net BA8: now also U3.49 (IO_33); no longer U3.23 (IO_75)
- net BA9: now also U3.47 (IO_31); no longer U3.24 (IO_76)
- net BnW: now also U3.8 (IO_7); no longer U3.37 (IO_24)
- net LA0: now also U3.57 (IO_40); no longer U3.93 (IO_64)
- net LA1: now also U3.56 (IO_39); no longer U3.94 (IO_65)
- net LS0: now also U3.67 (IO_47); no longer U3.13 (IO_11)
- net LS1: now also U3.65 (IO_46); no longer U3.12 (IO_10)
- net LS2: now also U3.64 (IO_45); no longer U3.10 (IO_9)
- net LS3: now also U3.63 (IO_44); no longer U3.9 (IO_8)
- net PCA0: now also U3.10 (IO_9); no longer U3.65 (IO_46)
- net PCA1: now also U3.12 (IO_10); no longer U3.67 (IO_47)
- net PCA2: now also U3.13 (IO_11); no longer U3.68 (IO_48)
- net PCA3: now also U3.14 (IO_12); no longer U3.69 (IO_49)
- net PCA4: now also U3.16 (IO_13); no longer U3.70 (IO_50)
- net PCA5: now also U3.17 (IO_14); no longer U3.71 (IO_51)
- net PCA6: now also U3.19 (IO_71); no longer U3.72 (IO_52)
- net PCA7: now also U3.20 (IO_72); no longer U3.75 (IO_53)
- net PCA8: now also U3.21 (IO_73); no longer U3.76 (IO_54)
- net PCA9: now also U3.22 (IO_74); no longer U3.77 (IO_55)
- net PCD0: now also U3.81 (IO_59); no longer U3.64 (IO_45)
- net RAMnPROM: now also U3.78 (IO_56); no longer U3.28 (IO_16)
- net RnW: now also U3.33 (IO_21); no longer U3.40 (IO_25)
- net SN0: now also U3.7 (IO_6); no longer U3.58 (IO_41)
- net SN1: now also U3.6 (IO_5); no longer U3.57 (IO_40)
- net SN2: now also U3.5 (IO_4); no longer U3.56 (IO_39)
- net SN3: now also U3.2 (IO_3); no longer U3.55 (IO_38)
- net SN4: now also U3.60 (IO_42); no longer U3.54 (IO_37)
- net SN5: now also U3.61 (IO_43); no longer U3.53 (IO_36)
- net SN6: now also U3.58 (IO_41); no longer U3.52 (IO_35)
- net ST0: now also U3.1 (IO_2); no longer U3.27 (IO_15)
- net ST1: now also U3.100 (IO_70); no longer U3.17 (IO_14)
- net ST2: now also U3.99 (IO_69); no longer U3.16 (IO_13)
- net ST3: now also U3.98 (IO_68); no longer U3.14 (IO_12)
- net /ADDR2: now also U3.96 (IO_66); no longer U3.50 (IO_34)
- net /AEN: now also U3.31 (IO_19); no longer U3.60 (IO_42)
- net /AS: now also U3.9 (IO_8); no longer U3.35 (IO_22)
- net /BHE: now also U3.24 (IO_76); no longer U3.31 (IO_19)
- net /BLE: now also U3.25 (IO); no longer U3.32 (IO_20)
- net /CS_2716: now also U3.29 (IO_17); no longer U3.48 (IO_32)
- net /CS_RAM: now also U3.28 (IO_16); no longer U3.49 (IO_33)
- net /DS: now also U3.97 (IO_67); no longer U3.36 (IO_23)
- net /HOLD: now also U3.36 (IO_23); no longer U3.44 (IO_28)
- net /IOR: now also U3.23 (IO_75); no longer U3.61 (IO_43)
- net /IOW: now also U3.27 (IO_15); no longer U3.63 (IO_44)
- net /MRD: now also U3.30 (IO_18); no longer U3.29 (IO_17)
- net /MREQ: now also U3.94 (IO_65); no longer U3.41 (IO_26)
- net /MWR: now also U3.55 (IO_38); no longer U3.30 (IO_18)
- net /NMI: now also U3.93 (IO_64); no longer U3.85 (IO_62)
- net /OE_6116: now also U3.42 (IO_27); no longer U3.45 (IO_29)
- net /PC: now also U3.52 (IO_35); no longer U3.46 (IO_30)
- net /WE: now also U3.45 (IO_29); no longer U3.42 (IO_27)
- net /Z: now also U3.53 (IO_36); no longer U3.47 (IO_31)
- new net GND: C1.2, C10.2, C11.2, C12.2, C13.2, C14.2, C15.2, C16.2, C17.2, C18.2, C19.2, C2.2, C20.2, C21.2, C22.2, C23.2, C24.2, C3.2, C4.2, C5.2, C6.2, C7.2, C8.2, C9.2, J1.10 (Pin_10), J1.2 (Pin_2), P1.B1 (GND), P1.B10 (GND), P1.B31 (GND), TEST-PDS1.2 (Pin_2), TEST-PDS2.2 (Pin_2), U1.36 (GND), U12.10 (GND), U13.10 (GND), U2.12 (VSS), U2.34 (VSS), U3.11 (GNDIO_3), U3.26 (GNDIO), U3.38 (GNDINT), U3.43 (GNDIO_2), U3.59 (GNDIO_5), U3.74 (GNDIO_6), U3.86 (GNDINT_2), U3.95 (GNDIO_4), U4.12 (GND), U5.1 (OE), U5.10 (GND), U6.1 (OE), U6.10 (GND), U7.12 (GND), U8.12 (GND), U9.14 (GND), U9.4 (/INH)

Commit message: Add files via upload
Updates on component fields to generate BOM
Parts:
- C1, C10, C13, C18, C21, C24, C4, C7: PACKAGE (none) -> "0805"
- C11, C12, C14, C15, C16, C17, C19, C2, C20, C22, C23, C3, C5, C6, C8, C9, R1, R10, R11, R12, R13, R14, R15, R16, R17, R18, R19, R2, R20, R21, R22, R23, R24, R25, R26, R27, R28, R29, R3, R30, R31, R32, R33, R4, R5, R6, R7, R8, R9: PACKAGE (none) -> "0603"
- J1: SUPPLIER (none) -> Digikey, AliExpress, eBay
- LOGO1, P1, U11: now left out of the parts list
- U1: PACKAGE (none) -> DIP-48; SUPPLIER (none) -> eBay
- U12, U13, U5, U6: PACKAGE (none) -> DIP-20; SUPPLIER (none) -> Digikey, AliExpress, eBay
- U2: Manufacturer (none) -> Infineon; PACKAGE (none) -> TSOP-II-44; SUPPLIER (none) -> Digikey; SUPPLIER2 (none) -> Farnell UK; Supplier Part Number (none) -> 448-CY62157ELL-45ZSXI-ND; Supplier2 Part Number (none) -> 2767919
- U3: Manufacturer (none) -> Altera/Intel; SUPPLIER ALTERA -> AliExpress, eBay
- U4: PACKAGE (none) -> DIP-24; SUPPLIER (none) -> eBay, AliExpress
- U7: PACKAGE (none) -> DIP-24; SUPPLIER (none) -> AliExpress, eBay
- U8: PACKAGE (none) -> DIP-24; SUPPLIER (none) -> Digikey, AliExpress, eBay
- U9: PACKAGE (none) -> DIP-18; SUPPLIER (none) -> AliExpress, eBay
- Y1: PACKAGE (none) -> HC49-U; SUPPLIER (none) -> Digikey, AliExpress
